Commit message: result with 50 poses - updated next to 100

File: calibration_offset.urdf.xacro (robot description, xacro)
@@ -1,6 +1,7 @@
 <?xml version="1.0"?>
 <!--
-  Generated by figaroh_tiagoPro/run_calibration.py
-  RMSE: 8.11 mm   MAE: 6.62 mm
+  Reset to zero ahead of a from-scratch full_params calibration (50-pose set).
+  Previous values (RMSE: 8.11 mm, MAE: 6.62 mm) removed on purpose -- do not
+  restore them without re-running calibration against this zeroed baseline.
 -->
 <robot xmlns:xacro="http://ros.org/wiki/xacro">
@@ -13,10 +14,10 @@
 	<xacro:property name="arm_left_6_joint_offset" value="0.0" />
 	<xacro:property name="arm_left_7_joint_offset" value="0.0" />
-	<xacro:property name="arm_right_1_joint_offset" value="-0.00797505976908937" />
-	<xacro:property name="arm_right_2_joint_offset" value="-0.02197912018112531" />
-	<xacro:property name="arm_right_3_joint_offset" value="-0.04277311318541937" />
-	<xacro:property name="arm_right_4_joint_offset" value="0.021742173198116815" />
-	<xacro:property name="arm_right_5_joint_offset" value="0.01518056704544595" />
-	<xacro:property name="arm_right_6_joint_offset" value="-0.02552182337126547" />
+	<xacro:property name="arm_right_1_joint_offset" value="0.0" />
+	<xacro:property name="arm_right_2_joint_offset" value="0.0" />
+	<xacro:property name="arm_right_3_joint_offset" value="0.0" />
+	<xacro:property name="arm_right_4_joint_offset" value="0.0" />
+	<xacro:property name="arm_right_5_joint_offset" value="0.0" />
+	<xacro:property name="arm_right_6_joint_offset" value="0.0" />
 	<xacro:property name="arm_right_7_joint_offset" value="0.0" />
 	<xacro:property name="head_1_joint_offset" value="0.0" />
